Commit message: Lidar Sensor updated

File: src/robot_description/urdf/simple_robot.urdf (robot description, URDF)
Before this commit: robot simple_robot, 3 links, 2 joints
Links:
- added link lidar_link; visual cylinder length=0.1 radius=0.05
Joints:
- added joint lidar_joint: type fixed, parent base_link, child lidar_link, origin xyz=0 0 0.1 rpy=0 0 0

File: src/robot_description/urdf/simple_robot.xacro (robot description, xacro)
@@ -1,5 +1,5 @@
 <robot name="simple_robot" xmlns:xacro="http://www.ros.org/wiki/xacro">
-#using xacro macro for wheels only because code is same for wheels
-#from xacro only...macro files can be created
+<!-- using xacro macro for wheels only because code is same for wheels -->
+<!-- from xacro only...macro files can be created -->
 <xacro:property name="wheel_radius" value="0.1"/>
 <xacro:property name="wheel_width" value="0.05"/>
@@ -35,3 +35,15 @@
 <xacro:wheel name="left_wheel" y_offset="${wheel_offset}"/>
 <xacro:wheel name="right_wheel" y_offset="-${wheel_offset}"/>
+<link name="lidar_link">
+    <visual>
+        <geometry>
+            <cylinder length="0.1" radius="0.05"/>
+        </geometry>
+    </visual>
+</link>
+<joint name="lidar_joint" type="fixed">
+    <parent link="base_link"/>
+    <child link="lidar_link"/>
+    <origin xyz="0 0 0.1" rpy="0 0 0"/>
+</joint>
 </robot>

Commit message: Camera link added

File: src/robot_description/urdf/simple_robot.urdf (robot description, URDF)
Before this commit: robot simple_robot, 4 links, 3 joints
Links:
- added link camera_link; visual box size=0.1 0.1 0.05
- added link camera_optical_frame; visual box size=0.1 0.1 0.05
Joints:
- added joint camera_joint: type fixed, parent base_link, child camera_link, origin xyz=0 0 0.1 rpy=0 0 0
- added joint camera_optical_frame_joint: type fixed, parent camera_link, child camera_optical_frame, origin xyz=0 0 0.1 rpy=0 0 0

File: src/robot_description/urdf/simple_robot.xacro (robot description, xacro)
@@ -23,5 +23,7 @@
                 <cylinder radius="${wheel_radius}" length="${wheel_width}"/>
             </geometry>
-            <material name="black"/>
+            <material name="black">
+                <color rgba="0 0 0 1"/>
+            </material>
         </visual>
     </link>
@@ -47,3 +49,27 @@
     <origin xyz="0 0 0.1" rpy="0 0 0"/>
 </joint>
+<link name="camera_link">
+    <visual>
+        <geometry>
+            <box size="0.1 0.1 0.05"/>
+        </geometry>
+    </visual>
+</link>
+<joint name="camera_joint" type="fixed">
+    <parent link="base_link"/>
+    <child link="camera_link"/>
+    <origin xyz="0 0 0.1" rpy="0 0 0"/>
+</joint>
+<link name="camera_optical_frame">
+    <visual>
+        <geometry>
+            <box size="0.1 0.1 0.05"/>
+        </geometry>
+    </visual>
+</link>
+<joint name="camera_optical_frame_joint" type="fixed">
+    <parent link="camera_link"/>
+    <child link="camera_optical_frame"/>
+    <origin xyz="0 0 0.1" rpy="0 0 0"/>
+</joint>
 </robot>

Commit message: launch file

File: src/robot_description/urdf/simple_robot.urdf (robot description, URDF)
Before this commit: robot simple_robot, 6 links, 5 joints
Links:
- link base_link: mass None -> 5.0; geometry collision box size=0.5 0.4 0.1; visual box size=0.5 0.4 0.1
- link camera_optical_frame: geometry 
- link left_wheel: mass None -> 1.0; geometry collision cylinder length=0.05 radius=0.1; visual cylinder length=0.05 radius=0.1
- link right_wheel: mass None -> 1.0; geometry collision cylinder length=0.05 radius=0.1; visual cylinder length=0.05 radius=0.1
Joints:
- joint camera_joint: origin xyz=0 0 0.1 rpy=0 0 0 -> xyz=0.15 0 0.1 rpy=0 0 0
- joint camera_optical_frame_joint: origin xyz=0 0 0.1 rpy=0 0 0 -> xyz=0 0 0 rpy=-1.5708 0 -1.5708
- joint left_wheel_joint: origin xyz=0.0 0.225 -0.05 rpy=0 0 0 -> xyz=0 0.225 -0.05 rpy=0 0 0
- joint right_wheel_joint: origin xyz=0.0 -0.225 -0.05 rpy=0 0 0 -> xyz=0 -0.225 -0.05 rpy=0 0 0

File: src/robot_description/urdf/simple_robot.xacro (robot description, xacro)
@@ -5,15 +5,25 @@
 <xacro:property name="wheel_width" value="0.05"/>
 <xacro:property name="wheel_offset" value="0.225"/>
-<link name="base_link">
+  <link name="base_link">
     <visual>
-        <origin xyz="0 0 0" rpy="0 0 0"/>
-        <geometry>
-            <box size="0.5 0.4 0.1"/>
-        </geometry>
-        <material name="blue">
-            <color rgba="0 0 1 1"/>
-        </material>
+      <geometry>
+        <box size="0.5 0.4 0.1"/>
+      </geometry>
+      <material name="blue"/>
     </visual>
-</link>
+    <collision>
+      <geometry>
+        <box size="0.5 0.4 0.1"/>
+      </geometry>
+    </collision>
+    <inertial>
+      <mass value="5.0"/>
+      <inertia ixx="0.5" iyy="0.5" izz="0.5"
+              ixy="0.0" ixz="0.0" iyz="0.0"/>
+    </inertial>
+  </link>
+  <gazebo reference="base_link">
+    <material>Gazebo/Blue</material>
+  </gazebo>
 <xacro:macro name="wheel" params="name y_offset">
     <link name="${name}">
@@ -27,9 +37,20 @@
             </material>
         </visual>
+        <collision>
+            <origin xyz="0 0 0" rpy="1.5708 0 0"/>
+            <geometry>
+                <cylinder radius="${wheel_radius}" length="${wheel_width}"/>
+            </geometry>
+        </collision>
+        <inertial>
+            <mass value="1.0"/>
+            <inertia ixx="0.01" iyy="0.01" izz="0.01"
+                     ixy="0.0" ixz="0.0" iyz="0.0"/>
+        </inertial>
     </link>
     <joint name="${name}_joint" type="continuous">
         <parent link="base_link"/>
         <child link="${name}"/>
-        <origin xyz="0.0 ${y_offset} -0.05" rpy="0 0 0"/>
+        <origin xyz="0 ${y_offset} -0.05" rpy="0 0 0"/>
         <axis xyz="0 1 0"/>
     </joint>
@@ -59,17 +80,11 @@
     <parent link="base_link"/>
     <child link="camera_link"/>
-    <origin xyz="0 0 0.1" rpy="0 0 0"/>
+    <origin xyz="0.15 0 0.1" rpy="0 0 0"/>
 </joint>
-<link name="camera_optical_frame">
-    <visual>
-        <geometry>
-            <box size="0.1 0.1 0.05"/>
-        </geometry>
-    </visual>
-</link>
+<link name="camera_optical_frame"/>
 <joint name="camera_optical_frame_joint" type="fixed">
     <parent link="camera_link"/>
     <child link="camera_optical_frame"/>
-    <origin xyz="0 0 0.1" rpy="0 0 0"/>
+    <origin xyz="0 0 0" rpy="-1.5708 0 -1.5708"/>
 </joint>
 </robot>

Commit message: Add Gazebo simulation world and update robot description

File: src/robot_description/urdf/simple_robot.urdf (robot description, URDF)
Before this commit: robot simple_robot, 6 links, 5 joints
Links:
- added link front_caster, mass 0.5; collision sphere radius=0.05; visual sphere radius=0.05
- added link lidar_spinner_link, mass 0.05; visual cylinder length=0.12 radius=0.052
- added link rear_caster, mass 0.5; collision sphere radius=0.05; visual sphere radius=0.05
- link camera_link: mass None -> 0.3; geometry collision box size=0.1 0.05 0.05; visual box size=0.1 0.05 0.05
- link lidar_link: mass None -> 0.5; geometry collision cylinder length=0.1 radius=0.05; visual cylinder length=0.1 radius=0.05
Joints:
- removed joint camera_optical_frame_joint
- added joint camera_optical_joint: type fixed, parent camera_link, child camera_optical_frame, origin xyz=0 0 0 rpy=-1.5708 0 -1.5708
- added joint front_caster_joint: type fixed, parent base_link, child front_caster, origin xyz=0.2 0 -0.1
- added joint lidar_spinner_joint: type continuous, parent lidar_link, child lidar_spinner_link, origin xyz=0 0 0, axis 0 0 1
- added joint rear_caster_joint: type fixed, parent base_link, child rear_caster, origin xyz=-0.2 0 -0.1
- joint camera_joint: origin xyz=0.15 0 0.1 rpy=0 0 0 -> xyz=0.10 0 0.05
- joint left_wheel_joint: origin xyz=0 0.225 -0.05 rpy=0 0 0 -> xyz=0 0.225 -0.05
- joint lidar_joint: origin xyz=0 0 0.1 rpy=0 0 0 -> xyz=0 0 0.10
- joint right_wheel_joint: origin xyz=0 -0.225 -0.05 rpy=0 0 0 -> xyz=0 -0.225 -0.05

File: src/robot_description/urdf/simple_robot.xacro (robot description, xacro)
@@ -1,8 +1,22 @@
+<?xml version="1.0"?>
 <robot name="simple_robot" xmlns:xacro="http://www.ros.org/wiki/xacro">
-<!-- using xacro macro for wheels only because code is same for wheels -->
-<!-- from xacro only...macro files can be created -->
-<xacro:property name="wheel_radius" value="0.1"/>
-<xacro:property name="wheel_width" value="0.05"/>
-<xacro:property name="wheel_offset" value="0.225"/>
+  <!-- ================= PARAMETERS ================= -->
+  <xacro:property name="wheel_radius" value="0.1"/>
+  <xacro:property name="wheel_width" value="0.05"/>
+  <xacro:property name="wheel_offset_y" value="0.225"/>
+  <!-- ================= MATERIALS ================= -->
+  <material name="blue">
+    <color rgba="0 0 1 1"/>
+  </material>
+  <material name="black">
+    <color rgba="0 0 0 1"/>
+  </material>
+  <material name="red">
+    <color rgba="1 0 0 1"/>
+  </material>
+  <material name="green">
+    <color rgba="0 1 0 1"/>
+  </material>
+  <!-- ================= BASE LINK ================= -->
   <link name="base_link">
     <visual>
@@ -26,65 +40,249 @@
     <material>Gazebo/Blue</material>
   </gazebo>
-<xacro:macro name="wheel" params="name y_offset">
+  <!-- ================= WHEEL MACRO ================= -->
+  <xacro:macro name="wheel" params="name y_offset">
     <link name="${name}">
-        <visual>
-            <origin xyz="0 0 0" rpy="1.5708 0 0"/>
-            <geometry>
-                <cylinder radius="${wheel_radius}" length="${wheel_width}"/>
-            </geometry>
-            <material name="black">
-                <color rgba="0 0 0 1"/>
-            </material>
-        </visual>
-        <collision>
-            <origin xyz="0 0 0" rpy="1.5708 0 0"/>
-            <geometry>
-                <cylinder radius="${wheel_radius}" length="${wheel_width}"/>
-            </geometry>
-        </collision>
-        <inertial>
-            <mass value="1.0"/>
-            <inertia ixx="0.01" iyy="0.01" izz="0.01"
-                     ixy="0.0" ixz="0.0" iyz="0.0"/>
-        </inertial>
+      <visual>
+        <origin xyz="0 0 0" rpy="1.5708 0 0"/>
+        <geometry>
+          <cylinder radius="${wheel_radius}" length="${wheel_width}"/>
+        </geometry>
+        <material name="black"/>
+      </visual>
+      <collision>
+        <origin xyz="0 0 0" rpy="1.5708 0 0"/>
+        <geometry>
+          <cylinder radius="${wheel_radius}" length="${wheel_width}"/>
+        </geometry>
+      </collision>
+      <inertial>
+        <mass value="1.0"/>
+        <inertia ixx="0.1" iyy="0.1" izz="0.1"
+                ixy="0.0" ixz="0.0" iyz="0.0"/>
+      </inertial>
     </link>
     <joint name="${name}_joint" type="continuous">
-        <parent link="base_link"/>
-        <child link="${name}"/>
-        <origin xyz="0 ${y_offset} -0.05" rpy="0 0 0"/>
-        <axis xyz="0 1 0"/>
+      <parent link="base_link"/>
+      <child link="${name}"/>
+      <origin xyz="0 ${y_offset} -0.05"/>
+      <axis xyz="0 1 0"/>
     </joint>
-</xacro:macro>
-<xacro:wheel name="left_wheel" y_offset="${wheel_offset}"/>
-<xacro:wheel name="right_wheel" y_offset="-${wheel_offset}"/>
-<link name="lidar_link">
-    <visual>
-        <geometry>
-            <cylinder length="0.1" radius="0.05"/>
-        </geometry>
-    </visual>
-</link>
-<joint name="lidar_joint" type="fixed">
+    <gazebo reference="${name}">
+      <material>Gazebo/Black</material>
+      <mu1>1.5</mu1>
+      <mu2>1.5</mu2>
+      <kp>1000000</kp>
+      <kd>100</kd>
+    </gazebo>
+  </xacro:macro>
+  <!-- ================= CREATE WHEELS ================= -->
+  <xacro:wheel name="left_wheel" y_offset="${wheel_offset_y}"/>
+  <xacro:wheel name="right_wheel" y_offset="-${wheel_offset_y}"/>
+  <!-- ================= FRONT CASTER ================= -->
+  <link name="front_caster">
+    <visual>
+      <geometry>
+        <sphere radius="0.05"/>
+      </geometry>
+      <material name="black"/>
+    </visual>
+    <collision>
+      <geometry>
+        <sphere radius="0.05"/>
+      </geometry>
+    </collision>
+    <inertial>
+      <mass value="0.5"/>
+      <inertia ixx="0.001" iyy="0.001" izz="0.001"
+              ixy="0.0" ixz="0.0" iyz="0.0"/>
+    </inertial>
+  </link>
+  <joint name="front_caster_joint" type="fixed">
+    <parent link="base_link"/>
+    <child link="front_caster"/>
+    <origin xyz="0.2 0 -0.1"/>
+  </joint>
+  <gazebo reference="front_caster">
+    <material>Gazebo/Black</material>
+    <mu1>0.001</mu1>
+    <mu2>0.001</mu2>
+  </gazebo>
+  <!-- ================= REAR CASTER ================= -->
+  <link name="rear_caster">
+    <visual>
+      <geometry>
+        <sphere radius="0.05"/>
+      </geometry>
+      <material name="black"/>
+    </visual>
+    <collision>
+      <geometry>
+        <sphere radius="0.05"/>
+      </geometry>
+    </collision>
+    <inertial>
+      <mass value="0.5"/>
+      <inertia ixx="0.001" iyy="0.001" izz="0.001"
+              ixy="0.0" ixz="0.0" iyz="0.0"/>
+    </inertial>
+  </link>
+  <joint name="rear_caster_joint" type="fixed">
+    <parent link="base_link"/>
+    <child link="rear_caster"/>
+    <origin xyz="-0.2 0 -0.1"/>
+  </joint>
+  <gazebo reference="rear_caster">
+    <material>Gazebo/Black</material>
+    <mu1>0.001</mu1>
+    <mu2>0.001</mu2>
+  </gazebo>
+  <!-- ================= LIDAR ================= -->
+  <link name="lidar_link">
+    <visual>
+      <geometry>
+        <cylinder length="0.1" radius="0.05"/>
+      </geometry>
+      <material name="red"/>
+    </visual>
+    <collision>
+      <geometry>
+        <cylinder length="0.1" radius="0.05"/>
+      </geometry>
+    </collision>
+    <inertial>
+      <mass value="0.5"/>
+      <inertia ixx="0.01" iyy="0.01" izz="0.01"
+              ixy="0.0" ixz="0.0" iyz="0.0"/>
+    </inertial>
+  </link>
+  <link name="lidar_spinner_link">
+    <visual>
+      <geometry>
+        <cylinder length="0.12" radius="0.052"/>
+      </geometry>
+      <material name="red"/>
+    </visual>
+    <inertial>
+      <mass value="0.05"/>
+      <inertia ixx="0.0001" iyy="0.0001" izz="0.0001"
+              ixy="0.0" ixz="0.0" iyz="0.0"/>
+    </inertial>
+  </link>
+  <joint name="lidar_joint" type="fixed">
     <parent link="base_link"/>
     <child link="lidar_link"/>
-    <origin xyz="0 0 0.1" rpy="0 0 0"/>
-</joint>
-<link name="camera_link">
-    <visual>
-        <geometry>
-            <box size="0.1 0.1 0.05"/>
-        </geometry>
-    </visual>
-</link>
-<joint name="camera_joint" type="fixed">
+    <origin xyz="0 0 0.10"/>
+  </joint>
+  <joint name="lidar_spinner_joint" type="continuous">
+    <parent link="lidar_link"/>
+    <child link="lidar_spinner_link"/>
+    <origin xyz="0 0 0"/>
+    <axis xyz="0 0 1"/>
+  </joint>
+  <gazebo reference="lidar_link">
+    <material>Gazebo/Red</material>
+    <sensor name="lidar_sensor" type="gpu_lidar">
+      <always_on>true</always_on>
+      <visualize>true</visualize>
+      <update_rate>10</update_rate>
+      <topic>scan</topic>
+      <lidar>
+        <scan>
+          <horizontal>
+            <samples>720</samples>
+            <resolution>1</resolution>
+            <min_angle>-3.14159</min_angle>
+            <max_angle>3.14159</max_angle>
+          </horizontal>
+        </scan>
+        <range>
+          <min>0.1</min>
+          <max>10.0</max>
+          <resolution>0.01</resolution>
+        </range>
+      </lidar>
+    </sensor>
+  </gazebo>
+  <gazebo reference="lidar_spinner_link">
+    <material>Gazebo/Red</material>
+  </gazebo>
+  <gazebo>
+    <plugin
+      filename="gz-sim-joint-controller-system"
+      name="gz::sim::systems::JointController">
+      <joint_name>lidar_spinner_joint</joint_name>
+      <initial_velocity>3.0</initial_velocity>
+    </plugin>
+  </gazebo>
+  <!-- ================= DIFFERENTIAL DRIVE ================= -->
+  <gazebo>
+    <plugin
+      filename="gz-sim-diff-drive-system"
+      name="gz::sim::systems::DiffDrive">
+      <left_joint>left_wheel_joint</left_joint>
+      <right_joint>right_wheel_joint</right_joint>
+      <wheel_separation>0.4</wheel_separation>
+      <wheel_radius>0.1</wheel_radius>
+      <odom_topic>/odom</odom_topic>
+      <cmd_vel_topic>/cmd_vel</cmd_vel_topic>
+      <tf_topic>/tf</tf_topic>
+      <frame_id>odom</frame_id>
+      <child_frame_id>base_link</child_frame_id>
+      <odom_publish_frequency>50</odom_publish_frequency>
+      <max_linear_velocity>1.0</max_linear_velocity>
+      <max_angular_velocity>2.0</max_angular_velocity>
+      <min_linear_velocity>-1.0</min_linear_velocity>
+      <min_angular_velocity>-2.0</min_angular_velocity>
+      <max_linear_acceleration>1.0</max_linear_acceleration>
+      <max_angular_acceleration>2.0</max_angular_acceleration>
+    </plugin>
+  </gazebo>
+  <!-- ================= CAMERA ================= -->
+  <link name="camera_link">
+    <visual>
+      <geometry>
+        <box size="0.1 0.05 0.05"/>
+      </geometry>
+      <material name="green"/>
+    </visual>
+    <collision>
+      <geometry>
+        <box size="0.1 0.05 0.05"/>
+      </geometry>
+    </collision>
+    <inertial>
+      <mass value="0.3"/>
+      <inertia ixx="0.01" iyy="0.01" izz="0.01"
+              ixy="0.0" ixz="0.0" iyz="0.0"/>
+    </inertial>
+  </link>
+  <joint name="camera_joint" type="fixed">
     <parent link="base_link"/>
     <child link="camera_link"/>
-    <origin xyz="0.15 0 0.1" rpy="0 0 0"/>
-</joint>
-<link name="camera_optical_frame"/>
-<joint name="camera_optical_frame_joint" type="fixed">
+    <origin xyz="0.10 0 0.05"/>
+  </joint>
+  <gazebo reference="camera_link">
+    <material>Gazebo/Green</material>
+    <sensor type="camera" name="camera_sensor">
+      <always_on>true</always_on>
+      <update_rate>30</update_rate>
+      <visualize>true</visualize>
+      <topic>/camera/image_raw</topic>
+      <camera>
+        <horizontal_fov>1.396</horizontal_fov>
+        <image>
+          <width>640</width>
+          <height>480</height>
+          <format>R8G8B8</format>
+        </image>
+      </camera>
+    </sensor>
+  </gazebo>
+  <!-- ================= CAMERA OPTICAL FRAME ================= -->
+  <link name="camera_optical_frame"/>
+  <joint name="camera_optical_joint" type="fixed">
     <parent link="camera_link"/>
     <child link="camera_optical_frame"/>
     <origin xyz="0 0 0" rpy="-1.5708 0 -1.5708"/>
-</joint>
+  </joint>
 </robot>
